Commit message: Adding SICK LM200 to robot model

File: catkin_ws/src/building_mapper/urdf/sick_lm2xx.urdf.xacro (robot description, xacro)
@@ -1,2 +1,36 @@
 <robot>
+  <link name="sick_lm200-lm291_mount">
+    <visual>
+      <origin xyz="0 0 0" rpy="0 0 ${PI/2}"/>
+      <geometry>
+        <mesh filename="package://building_mapper/urdf/meshes/SICK_LM200-LM291_MOUNT.stl" scale="0.001 0.001 0.001"/>
+      </geometry>
+      <material name="black"/>
+    </visual>
+  </link>
+  <joint name="sick_lm200-lm291_mount_joint" type="fixed">
+    <parent link="chassis_link"/>
+    <child link="sick_lm200-lm291_mount"/>
+    <origin xyz="0.0295 0 0.18" rpy="0 0 0"/>
+  </joint>
+  <link name="sick_lm200-lm291">
+    <visual>
+      <origin xyz="0 0 0" rpy="0 0 ${PI/2}"/>
+      <geometry>
+        <mesh filename="package://building_mapper/urdf/meshes/SICK_LM200-LM291.stl" scale="0.001 0.001 0.001"/>
+      </geometry>
+      <material name="blue">
+        <color rgba="0.25 0.55 1.0 1.0"/>
+      </material>
+    </visual>
+    <inertial>
+      <mass value="4.5"/>
+      <inertia ixx="0.3136" ixy="-0.0008" ixz="0.0164" iyy="0.3922" iyz="-0.0009" izz="0.4485"/>
+    </inertial>
+  </link>
+  <joint name="sick_lm2xx_lidar_joint" type="fixed">
+    <parent link="sick_lm200-lm291_mount"/>
+    <child link="sick_lm200-lm291"/>
+    <origin xyz="0.0935 0 0.079" rpy="0 0 0"/>
+  </joint>
 </robot>

Commit message: Updating all launch files to use sick, when approprite, and URDF file to use the correct frame id.

File: catkin_ws/src/building_mapper/urdf/sick_lm2xx.urdf.xacro (robot description, xacro)
@@ -1,4 +1,4 @@
 <robot>
-  <link name="sick_lm200-lm291_mount">
+  <link name="laser_mount">
     <visual>
       <origin xyz="0 0 0" rpy="0 0 ${PI/2}"/>
@@ -11,8 +11,8 @@
   <joint name="sick_lm200-lm291_mount_joint" type="fixed">
     <parent link="chassis_link"/>
-    <child link="sick_lm200-lm291_mount"/>
+    <child link="laser_mount"/>
     <origin xyz="0.0295 0 0.18" rpy="0 0 0"/>
   </joint>
-  <link name="sick_lm200-lm291">
+  <link name="laser">
     <visual>
       <origin xyz="0 0 0" rpy="0 0 ${PI/2}"/>
@@ -28,8 +28,29 @@
       <inertia ixx="0.3136" ixy="-0.0008" ixz="0.0164" iyy="0.3922" iyz="-0.0009" izz="0.4485"/>
     </inertial>
+    <sensor type="ray" name="sick_lm200-lm291">
+      <!-- <update_rate>75</update_rate>
+      <ray>
+        <horizontal>
+          <samples>361</samples>
+          <resolution>1</resolution>
+          <min_angle>{-PI/2}</min_angle>
+          <max_angle>{PI/2}</max_angle>
+        </horizontal>
+        <range>
+          <min>0.10</min>
+          <max>30.0</max>
+          <resolution>0.01</resolution>
+        </range>
+        <noise>
+          <type>gaussian</type>
+          <mean>0.0</mean>
+          <stddev>0.001</stddev>
+        </noise>
+      </ray> -->
+    </sensor>
   </link>
   <joint name="sick_lm2xx_lidar_joint" type="fixed">
-    <parent link="sick_lm200-lm291_mount"/>
-    <child link="sick_lm200-lm291"/>
+    <parent link="laser_mount"/>
+    <child link="laser"/>
     <origin xyz="0.0935 0 0.079" rpy="0 0 0"/>
   </joint>

Commit message: Updating URDF inertia values.

File: catkin_ws/src/building_mapper/urdf/sick_lm2xx.urdf.xacro (robot description, xacro)
@@ -1,3 +1,6 @@
 <robot>
+  <material name="blue">
+    <color rgba="0.25 0.55 1.0 1.0"/>
+  </material>
   <link name="laser_mount">
     <visual>
@@ -14,4 +17,7 @@
     <origin xyz="0.0295 0 0.18" rpy="0 0 0"/>
   </joint>
+  <gazebo reference="laser_mount">
+    <material name="black"/>
+  </gazebo>
   <link name="laser">
     <visual>
@@ -20,11 +26,9 @@
         <mesh filename="package://building_mapper/urdf/meshes/SICK_LM200-LM291.stl" scale="0.001 0.001 0.001"/>
       </geometry>
-      <material name="blue">
-        <color rgba="0.25 0.55 1.0 1.0"/>
-      </material>
+      <material name="blue"/>
     </visual>
     <inertial>
       <mass value="4.5"/>
-      <inertia ixx="0.3136" ixy="-0.0008" ixz="0.0164" iyy="0.3922" iyz="-0.0009" izz="0.4485"/>
+      <inertia ixx="0.025664" ixy="0.0" ixz="0.0" iyy="0.018135" iyz="0.0" izz="0.025547"/>
     </inertial>
     <sensor type="ray" name="sick_lm200-lm291">
@@ -55,3 +59,6 @@
     <origin xyz="0.0935 0 0.079" rpy="0 0 0"/>
   </joint>
+  <gazebo reference="laser">
+    <material name="blue"/>
+  </gazebo>
 </robot>

Commit message: Updating transform to use front_mount as the parrent instead of chassis_link.

File: catkin_ws/src/building_mapper/urdf/sick_lm2xx.urdf.xacro (robot description, xacro)
@@ -13,7 +13,7 @@
   </link>
   <joint name="sick_lm200-lm291_mount_joint" type="fixed">
-    <parent link="chassis_link"/>
+    <parent link="front_mount"/>
     <child link="laser_mount"/>
-    <origin xyz="0.0295 0 0.18" rpy="0 0 0"/>
+    <origin xyz="-0.091 0 0" rpy="0 0 0"/>
   </joint>
   <gazebo reference="laser_mount">
